File: kicad/rc-low-pass.kicad_pcb (KiCad board)
At the start: 2 copper layers, 54.4 x 48.3 mm, 11 parts, among them J1 Out, SW1 LEVEL 1, SW2 LEVEL 2, SW3 LEVEL 3

Commit message: add input voltage
Parts:
- added J2: In, TerminalBlock_Phoenix:TerminalBlock_Phoenix_MKDS-1,5-2-5.08_1x02_P5.08mm_Horizontal, F.Cu at (166.4, 78.3)
- moved SW1 8.93 mm to (160.8, 86.2)
- moved SW2 6.31 mm to (160.8, 95.5)
- moved R3 4.65 mm to (154.9, 95.4)
- moved SW3 3.82 mm to (160.8, 104.7)
- moved R2 3.65 mm to (154.8, 112.1)
- renumbered 2K to R2, 2K to R3
Connections:
- A1 pad 30: unconnected-(A1-Pad30) -> VOLTAGE_IN
Routing:
- net GND1: track 21.1 -> 42.9 mm
- net VOLTAGE_IN: track 0.00 -> 13.9 mm
- net ANALOG: track 62.1 -> 53.9 mm
- net Net-(R2-Pad2): track 18.7 -> 16.8 mm
Other:
- board text added: "5-12v"

Commit message: add led indicators of levels
Parts:
- added D1: LEVEL 1, LED_THT:LED_D5.0mm, F.Cu at (111.3, 106.6)
- added D2: LEVEL 2, LED_THT:LED_D5.0mm, F.Cu at (118.7, 106.6)
- added D3: LEVEL 3, LED_THT:LED_D5.0mm, F.Cu at (126.1, 106.5)
- added R4: 220, Resistor_THT:R_Axial_DIN0411_L9.9mm_D3.6mm_P12.70mm_Horizontal, F.Cu at (112.5, 88.3)
- added R5: 220, Resistor_THT:R_Axial_DIN0411_L9.9mm_D3.6mm_P12.70mm_Horizontal, F.Cu at (117.6, 88.2)
- added R6: 220, Resistor_THT:R_Axial_DIN0411_L9.9mm_D3.6mm_P12.70mm_Horizontal, F.Cu at (123.0, 88.4)
- moved C1 17.3 mm to (126.8, 77.6), turned to 90 degrees
- moved H1 7.91 mm to (113.2, 114.9)
- moved J1 7.90 mm to (119.2, 80.1)
- moved R1 0.89 mm to (128.3, 101.0)
Connections:
- A1 pad 5: unconnected-(A1-Pad5) -> LED_1
- A1 pad 6: unconnected-(A1-Pad6) -> LED_2
- A1 pad 7: unconnected-(A1-Pad7) -> LED_3
Routing:
- net GND: track 27.6 -> 72.1 mm
- net LED_1: track 0.00 -> 21.8 mm
- net LED_2: track 0.00 -> 17.7 mm
- net LED_3: track 0.00 -> 11.4 mm
- net Net-(R6-Pad2): track 0.00 -> 7.90 mm
- net Net-(R5-Pad2): track 0.00 -> 7.22 mm
- net Net-(R4-Pad2): track 0.00 -> 6.17 mm
- net VOLTAGE_OUT: track 16.4 -> 20.0 mm
- net ARDUINO_PIN: track 11.3 -> 9.64 mm
Other:
- board size 54.4 x 48.3 mm -> 62.9 x 48.3 mm

Commit message: code update
Parts:
- renumbered R2 to 2K, R3 to 2K
Changed lines of the file:
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@@
     (property "Sheetname" "")
     (attr through_hole)
-    (fp_text reference "R2" (at 6.45 0.1 90) (layer "F.SilkS")
+    (fp_text reference "2K" (at 6.45 0.1 90) (layer "F.SilkS")
       (effects (font (size 2 2) (thickness 0.3)))
     )
@@
     (property "Sheetname" "")
     (attr through_hole)
-    (fp_text reference "R3" (at 6.95 0.1 90) (layer "F.SilkS")
+    (fp_text reference "2K" (at 6.95 0.1 90) (layer "F.SilkS")
       (effects (font (size 2 2) (thickness 0.3)))
     )
